File: PAMI/PAMI 2025/PAMI 2025.kicad_sch (KiCad schematic)
At the start: 14 parts, among them M1 Motor_DC, M2 Motor_DC, M3 Motor_Servo

Commit message: adaptateur batterie
Connections:
- net at D1.3 (GA): no longer R5.1
- net at M3.1 (PWM): now also A1.14 (D11); no longer A1.16 (D13)
- net at R6.2: now also A1.16 (D13); no longer A1.14 (D11)
- net at R4.2: now also A1.10 (D7); no longer A1.12 (D9)
- net at R5.2: now also A1.11 (D8); no longer A1.13 (D10)
- net at M1.1 (+): now also A1.12 (D9); no longer A1.10 (D7)
- net at M1.2 (-): no longer A1.11 (D8)
Other:
- moved on the sheet: A1, D1, M3, R4, R5, R6

Commit message: code pami
Parts:
- renumbered blue/yellow to blue/yellow1, tirette- to tirette-1
Connections:
- net at D1.3 (GA): now also R5.1
Changed lines of the file:
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@@
-	(wire
-		(pts
-			(xy 81.28 121.92) (xy 81.28 123.19)
-		)
-		(stroke
-			(width 0)
-			(type default)
-		)
-	)
 	(wire
 		(pts
@@
 		(pts
 			(xy 87.63 127) (xy 115.57 127)
+		)
+		(stroke
+			(width 0)
+			(type default)
+		)
+	)
+	(wire
+		(pts
+			(xy 81.28 121.92) (xy 81.28 124.46)
 		)
 		(stroke
@@
 		(on_board yes)
 		(dnp no)
-		(property "Reference" "tirette-"
+		(property "Reference" "tirette-1"
 			(at 98.298 106.426 0)
 			(effects
@@
 			(project ""
 				(path "/9d7115ee-b553-46e9-9d14-4cd62ff89a57"
-					(reference "tirette-")
+					(reference "tirette-1")
 					(unit 1)
 				)
@@
 		(on_board yes)
 		(dnp no)
-		(property "Reference" "blue/yellow"
+		(property "Reference" "blue/yellow1"
 			(at 97.536 86.106 0)
 			(effects
@@
 			(project ""
 				(path "/9d7115ee-b553-46e9-9d14-4cd62ff89a57"
-					(reference "blue/yellow")
-					(unit 1)
-				)
+					(reference "blue/yellow1")
+					(unit 1)
+				)
